Commit message: lidar modify

File: src/mywaybot_gazebo/urdf/lidar.xacro (robot description, xacro)
@@ -1,4 +1,5 @@
 <?xml version="1.0"?>
 <robot xmlns:xacro="http://www.ros.org/wiki/xacro">
+<xacro:property name="M_PI" value="3.1415926535897931" />
 <gazebo reference="base_scan">
   <material>Gazebo/Red</material>
@@ -10,11 +11,11 @@
           <scan>
               <horizontal>
-                  <samples>4</samples>
-                  <min_angle>-3.14</min_angle>
-                  <max_angle>3.14</max_angle>
+                <samples>500</samples>
+                <min_angle>-1.57</min_angle>
+                <max_angle>1.57</max_angle>
               </horizontal>
           </scan>
           <range>
-              <min>0.3</min>
+              <min>0.05</min>
               <max>12</max>
           </range>

File: src/mywaybot_gazebo/urdf/mywaybot.xacro (robot description, xacro)
@@ -122,5 +122,5 @@
     </inertial>
     <visual>
-        <origin xyz="0 0 0" rpy="0 0 0" />
+        <origin xyz="0 0 0.0115" rpy="0 0 0" />
         <geometry>
             <mesh filename="file://$(find mywaybot_gazebo)/models/dae/laser.dae"  />
@@ -131,5 +131,5 @@
     </visual>
     <collision>
-        <origin xyz="0 0 0" rpy="0 0 0" />
+        <origin xyz="0 0 0.0115" rpy="0 0 0" />
         <geometry>
             <mesh filename="file://$(find mywaybot_gazebo)/models/dae/laser.dae"  />
@@ -138,14 +138,14 @@
     </link>
     <!-- JOINT-->
+    <joint name="base_joint" type="fixed">
+        <parent link="base_footprint" />
+        <child link="base_link" />
+        <origin xyz="0 0 0.010" rpy="0 0 0" />
+    </joint>
     <joint name="scan_joint" type="fixed">
-        <origin xyz="0.0405788546534533 0 0.0982633999999999" rpy="0 0 0" />
+        <origin xyz="0.0405788546534533 0 0.08676339999" rpy="0 0 0" />
         <parent link="base_link" />
         <child link="base_scan" />
         <axis xyz="0 0 0" />
-    </joint>
-     <joint name="base_joint" type="fixed">
-        <parent link="base_footprint" />
-        <child link="base_link" />
-        <origin xyz="0 0 0.010" rpy="0 0 0" />
     </joint>
     <joint name="wheel1_joint" type="continuous">

Commit message: fixed urdf

File: src/mywaybot_gazebo/urdf/lidar.xacro (robot description, xacro)
@@ -2,5 +2,5 @@
 <robot xmlns:xacro="http://www.ros.org/wiki/xacro">
 <xacro:property name="M_PI" value="3.1415926535897931" />
-<gazebo reference="base_scan">
+<gazebo reference="lidar_link">
   <material>Gazebo/Red</material>
   <sensor name="laser" type="ray">
@@ -23,8 +23,8 @@
       <plugin name="laser_controller" filename="libgazebo_ros_ray_sensor.so">
           <ros>
-              <argument>~/out:=scan</argument>
+              <remapping>~/out:=scan</remapping>
           </ros>
           <output_type>sensor_msgs/LaserScan</output_type>
-          <frame_name>laser_frame</frame_name>
+          <frame_name>lidar_link</frame_name>
       </plugin>
   </sensor>

File: src/mywaybot_gazebo/urdf/mywaybot.xacro (robot description, xacro)
@@ -131,5 +131,5 @@
     </collision>
     </link>
-    <link name="scan">
+    <link name="lidar_link">
     <inertial>
         <origin xyz="8.52131440630677E-05 -9.55220519319054E-05 0.0140146397972782" rpy="0 0 0" />
@@ -138,5 +138,5 @@
     </inertial>
     <visual>
-        <origin xyz="0 0 0" rpy="0 0 0" />
+        <origin xyz="0 0 -0.0298" rpy="0 0 0" />
         <geometry>
           <mesh filename="file://$(find mywaybot_gazebo)/models/stl/scan.stl"  />
@@ -147,5 +147,5 @@
     </visual>
     <collision>
-        <origin xyz="0 0 0" rpy="0 0 0" />
+        <origin xyz="0 0 -0.0298" rpy="0 0 0" />
         <geometry>
           <mesh filename="file://$(find mywaybot_gazebo)/models/stl/scan.stl"  />
@@ -160,5 +160,5 @@
     </inertial>
     <visual>
-        <origin xyz="0 0 0" rpy="0 0 0" />
+        <origin xyz="0 0 0" rpy="1.57 0 1.57" />
         <geometry>
             <mesh filename="file://$(find mywaybot_gazebo)/models/stl/imu.stl"  />
@@ -169,5 +169,5 @@
     </visual>
     <collision>
-        <origin xyz="0 0 0" rpy="0 0 0" />
+        <origin xyz="0 0 0" rpy="1.57 0 1.57" />
         <geometry>
             <mesh filename="file://$(find mywaybot_gazebo)/models/stl/imu.stl"  />
@@ -179,5 +179,5 @@
         <parent link="base_footprint" />
         <child link="base_link" />
-        <origin xyz="0 0 0.010" rpy="0 0 3.1416" />
+        <origin xyz="0 0 0.010" rpy="0 0 3.14" />
     </joint>
     <joint name="wheel1_joint" type="continuous">
@@ -206,11 +206,11 @@
     </joint>
     <joint name="scan_joint" type="fixed">
-        <origin xyz="-0.04 0 0.056963" rpy="0 0 3.1416" />
-        <parent link="base_link" />
-        <child link="scan" />
+        <origin xyz="-0.04 0 0.086763" rpy="0 0 3.14" />
+        <parent link="base_link" />
+        <child link="lidar_link" />
         <axis xyz="0 0 0" />
     </joint>
     <joint name="imu_joint" type="fixed">
-        <origin xyz="0.0499999999999996 -0.00999999999999986 0.0622634" rpy="1.5707963267949 0 1.5707963267949" />
+        <origin xyz="0.0499999999999996 -0.00999999999999986 0.0622634" rpy="0 0 3.14" />
         <parent link="base_link" />
         <child link="imu" />

File: src/mywaybot_gazebo/urdf/omni_drive.urdf.xacro (robot description, xacro)
@@ -3,13 +3,13 @@
     <plugin name="object_controller" filename="libgazebo_ros_planar_move.so">
       <ros>
-        <remapping>odom:=odom/unfiltered</remapping>
+        <remapping>odom:=odom</remapping>
       </ros>
       <command_topic>cmd_vel</command_topic>
-      <odometry_topic>odom/unfiltered</odometry_topic>
+      <odometry_topic>odom</odometry_topic>
       <odometry_frame>odom</odometry_frame>
       <odometry_rate>20.0</odometry_rate>
-      <robot_base_frame>base_link</robot_base_frame>
+      <robot_base_frame>base_footprint</robot_base_frame>
       <publish_odom>true</publish_odom>
-      <publish_odom_tf>false</publish_odom_tf>
+      <publish_odom_tf>true</publish_odom_tf>
     </plugin>
   </gazebo>
